File: ayx.kicad_pcb (KiCad board)
At the start: 2 copper layers, 18.5 x 37.1 mm, 35 parts, among them J2 SWD, U1 STM32F405RGTx, U2 AY-3-8912A Socket, U3 LP2985-3.3, U4 LP2985-3.3, Y1 16MHz

Commit message: Fix some errors
Parts:
- added J1: USART, ayx:USART, B.Cu at (147.8, 99.1)
Connections:
- R6 pad 2: A_CHA -> A_OUT_L
- R9 pad 2: A_CHC -> A_OUT_R
- U1 pad 20: A_CHA -> A_OUT_L
- U1 pad 21: A_CHC -> A_OUT_R
- U1 pad 57: GND -> ~AY_SEL
- U1 pad 59: GND -> ~AY_A9
Routing:
- net A_OUT_L: track 0.00 -> 19.9 mm, vias 0 -> 3
- net A_OUT_R: track 0.00 -> 18.0 mm, vias 0 -> 3
- net A_CHC: track 29.7 -> 13.2 mm, vias 3 -> 0
- net A_CHA: track 29.9 -> 13.5 mm, vias 3 -> 0
- net GND: track 51.7 -> 44.7 mm
- net USART_TX: track 0.00 -> 3.26 mm, vias 0 -> 1
- net USART_RX: track 0.00 -> 2.94 mm, vias 0 -> 1
- net IOA6: track 13.8 -> 15.4 mm
Other:
- outline, holes or cut-outs redrawn
