File: ayx.sch (KiCad schematic (older format))
At the start: 36 parts, among them J1 USART, J2 SWD, U1 STM32F405RGTx, U2 AY-3-8912A Socket, U3 LP2985-3.3, U4 LP2985-3.3, Y1 16MHz

Commit message: Fix some errors
Parts:
- J1: footprint Pin_Headers:Pin_Header_Straight_1x03_Pitch2.00mm -> ayx:USART; symbol ayx:Conn_01x03_Female -> Connector:Conn_01x02_Female
- U1: footprint Housings_QFP:LQFP-64_10x10mm_Pitch0.5mm -> Package_QFP:LQFP-64_10x10mm_P0.5mm
- U2: footprint Housings_DIP:DIP-28_W15.24mm -> DIL28
Connections:
- net A_CHA: no longer R6.2, U1.20 (PA4)
- net A_CHC: no longer R9.2, U1.21 (PA5)
- net GND: no longer J1.1 (Pin_1), U1.57 (PB5), U1.59 (PB7)
- net USART_RX: now also J1.1 (Pin_1); no longer J1.2 (Pin_2)
- net USART_TX: now also J1.2 (Pin_2); no longer J1.3 (Pin_3)
- new net A_OUT_L: R6.2, U1.20 (PA4)
- new net A_OUT_R: R9.2, U1.21 (PA5)
- new net ~AY_A9: U1.59 (PB7)
- new net ~AY_SEL: U1.57 (PB5)
- no-connect marks 18 -> 20
Changed lines of the file:
@@
 EESchema Schematic File Version 4
 LIBS:ayx-cache
-EELAYER 26 0
+EELAYER 29 0
 EELAYER END
 $Descr A4 11693 8268
@@
 F 0 "U1" H 4970 5320 50  0000 L CNN
 F 1 "STM32F405RGTx" H 5280 3570 50  0000 L CNN
-F 2 "Housings_QFP:LQFP-64_10x10mm_Pitch0.5mm" H 4970 1870 50  0001 R CNN
+F 2 "Package_QFP:LQFP-64_10x10mm_P0.5mm" H 4970 1870 50  0001 R CNN
 F 3 "" H 5570 3570 50  0001 C CNN
 	1    5570 3570
@@
 F 0 "U2" H 1890 1940 50  0000 L BNN
 F 1 "AY-3-8912A Socket" H 1890 1840 50  0000 L BNN
-F 2 "Housings_DIP:DIP-28_W15.24mm" H 1890 1940 50  0001 C CNN
+F 2 "DIL28" H 1890 1940 50  0001 C CNN
 F 3 "" H 1890 1790 60  0001 C CNN
 	1    1890 1790
@@
 Z80_D7
 Text GLabel 6270 2370 2    49   Output ~ 0
-A_CHA
+A_OUT_L
 Text GLabel 6270 2470 2    49   Output ~ 0
-A_CHC
-$Comp
-L ayx:Conn_01x03_Female J1
+A_OUT_R
+$Comp
+L Connector:Conn_01x02_Female J1
 U 1 1 5B73F06D
 P 1790 4620
-F 0 "J1" H 1790 4820 50  0000 C CNN
+F 0 "J1" H 1790 4742 50  0000 C CNN
 F 1 "USART" H 1790 4420 50  0000 C CNN
-F 2 "Pin_Headers:Pin_Header_Straight_1x03_Pitch2.00mm" H 1790 4620 50  0001 C CNN
-F 3 "" H 1790 4620 50  0001 C CNN
+F 2 "ayx:USART" H 1790 4620 50  0001 C CNN
+F 3 "~" H 1790 4620 50  0001 C CNN
 	1    1790 4620
 	1    0    0    -1
@@
 Text GLabel 1590 5150 0    49   Output ~ 0
 SWCLK
-Text GLabel 1590 4520 0    49   UnSpc ~ 0
-GND
 Text GLabel 1590 5250 0    49   UnSpc ~ 0
 GND
@@
 Connection ~ 5670 5490
 Connection ~ 5470 5490
-Text GLabel 2360 3800 2    49   Output ~ 0
+Text GLabel 2350 3800 2    49   Output ~ 0
 ~AY_A9
 $Comp
@@
 	0    1    1    0
 $EndComp
-Text GLabel 3040 4750 2    49   Input ~ 0
+Text GLabel 3040 4750 2    49   Output ~ 0
 A_CHB
-Text GLabel 3040 4910 2    49   Input ~ 0
+Text GLabel 3040 4910 2    49   Output ~ 0
 A_CHC
 Wire Wire Line
@@
 Wire Wire Line
 	2590 4910 2650 4910
-Text GLabel 3040 4590 2    49   Input ~ 0
+Text GLabel 3040 4590 2    49   Output ~ 0
 A_CHA
 Wire Wire Line
 	2950 4590 2990 4590
-Text GLabel 2560 4590 0    49   Output ~ 0
-A_CHA
+Text GLabel 2560 4590 0    49   Input ~ 0
+A_OUT_L
 Wire Wire Line
 	2650 4590 2560 4590
@@
 	0    1    1    0
 $EndComp
-Text GLabel 3040 5290 2    49   Input ~ 0
+Text GLabel 3040 5290 2    49   Output ~ 0
 A_CHB
-Text GLabel 3040 5450 2    49   Input ~ 0
+Text GLabel 3040 5450 2    49   Output ~ 0
 A_CHC
 Wire Wire Line
@@
 Wire Wire Line
 	2650 5290 2590 5290
-Text GLabel 3040 5130 2    49   Input ~ 0
+Text GLabel 3040 5130 2    49   Output ~ 0
 A_CHA
 Wire Wire Line
 	2950 5130 3040 5130
-Text GLabel 2560 5450 0    49   Output ~ 0
-A_CHC
+Text GLabel 2560 5450 0    49   Input ~ 0
+A_OUT_R
 Wire Wire Line
 	2650 5450 2560 5450
@@
 	0    1    1    0
 $EndComp
-Text GLabel 2360 3970 2    49   Output ~ 0
-~AY_SEL
 Wire Wire Line
 	5670 5370 5670 5490
@@
 Text GLabel 9300 1990 0    49   UnSpc ~ 0
 VDD5
-Text GLabel 2160 3800 0    49   UnSpc ~ 0
-GND
-Text GLabel 2160 3970 0    49   UnSpc ~ 0
-GND
-Wire Wire Line
-	2160 3800 2360 3800
-Wire Wire Line
-	2160 3970 2360 3970
 Text GLabel 5670 5670 3    49   UnSpc ~ 0
 GNDA
@@
 Wire Wire Line
 	2980 5450 3040 5450
+NoConn ~ 2150 3800
+NoConn ~ 2150 4000
+Text GLabel 2350 4000 2    49   Output ~ 0
+~AY_SEL
+Wire Wire Line
+	2150 4000 2350 4000
+Wire Wire Line
+	2150 3800 2350 3800
 $EndSCHEMATC
